File: Hardware/EDA/Arduino_Pro_Mini_mikroBUS.sch (KiCad schematic (older format))
At the start: 36 parts, among them CON1 BARREL_JACK, J1 HEADER_F_2.54MM_1R8P_ST_AU_PTH, J2 HEADER_F_2.54MM_1R8P_ST_AU_PTH, J3 HEADER_F_2.54MM_1R12P_ST_AU_P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, J4 HEADER_F_2.54MM_1R12P_ST_AU_P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, J5 Molex_0475710001, J6 HEADER_F_2.54MM_1R2P_ST_AU_PTH, M1 FID, M2 FID, M3 FID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

Commit message: Changed uSD CS pin to D10. Connected mikroBUS PWM pin to D6. Altered front silkscreen. Generated PDF schematic and Gerbers.
Connections:
- net labels removed: PWM
Other:
- moved on the sheet: B1, B2, C1, C2, C3, J5, LK1, M1, M2, M3, MH1, MH2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

Commit message: Removed barrel jack connector due to interference with Arduino Pro Mini. Updated schematic, layout and generated new gerbers. Added BOM file.
Parts:
- removed CON1: BARREL_JACK, Connect:Barrel_Jack_CUI_PJ-102AH, symbol BARREL_JACK
Connections:
- wire segments 140 -> 136
Other:
- moved on the sheet: P1
Changed lines of the file:
@@
 L HEADER_M_2.54MM_1R3P_ST_AU_PTH P1
 U 1 1 5A430131
-P 6800 6350
-F 0 "P1" H 6800 6550 40  0000 C CNN
-F 1 "HEADER_M_2.54MM_1R3P_ST_AU_PTH" V 6900 6350 40  0001 C CNN
-F 2 "Header:HEADER_M_2.54MM_1R3P_ST_AU_PTH" H 6800 6350 60  0001 C CNN
-F 3 "" H 6800 6350 60  0000 C CNN
-	1    6800 6350
+P 6800 5700
+F 0 "P1" H 6800 5900 40  0000 C CNN
+F 1 "HEADER_M_2.54MM_1R3P_ST_AU_PTH" V 6900 5700 40  0001 C CNN
+F 2 "Header:HEADER_M_2.54MM_1R3P_ST_AU_PTH" H 6800 5700 60  0001 C CNN
+F 3 "" H 6800 5700 60  0000 C CNN
+	1    6800 5700
 	1    0    0    -1
 $EndComp
-Text GLabel 6600 6350 0    40   Input ~ 0
+Text GLabel 6600 5700 0    40   Input ~ 0
 VCC
-Text GLabel 6600 6250 0    40   Input ~ 0
+Text GLabel 6600 5600 0    40   Input ~ 0
 5.0V
-Text GLabel 6600 6450 0    40   Input ~ 0
+Text GLabel 6600 5800 0    40   Input ~ 0
 3.3V
-Text Notes 6900 6450 0    60   ~ 0
+Text Notes 6900 5800 0    60   ~ 0
 VOLTAGE\nSELECT
 $Comp
@@
 Text Notes 4200 7250 1    60   ~ 0
 I2C
-$Comp
-L BARREL_JACK CON1
-U 1 1 5A43BDF7
-P 6700 5600
-F 0 "CON1" H 6700 5850 50  0000 C CNN
-F 1 "BARREL_JACK" H 6700 5400 50  0000 C CNN
-F 2 "Connect:Barrel_Jack_CUI_PJ-102AH" H 6700 5600 50  0001 C CNN
-F 3 "" H 6700 5600 50  0000 C CNN
-	1    6700 5600
-	1    0    0    -1
-$EndComp
-$Comp
-L GND #PWR014
-U 1 1 5A43C108
-P 7050 5750
-F 0 "#PWR014" H 7050 5500 50  0001 C CNN
-F 1 "GND" H 7050 5600 50  0001 C CNN
-F 2 "" H 7050 5750 50  0000 C CNN
-F 3 "" H 7050 5750 50  0000 C CNN
-	1    7050 5750
-	1    0    0    -1
-$EndComp
-Text GLabel 7100 5500 2    40   Input ~ 0
-RAW
 Text GLabel 7900 5550 1    40   Input ~ 0
 RAW
 $Comp
-L GND #PWR015
+L GND #PWR014
 U 1 1 5A43CC7D
 P 7900 5950
-F 0 "#PWR015" H 7900 5700 50  0001 C CNN
+F 0 "#PWR014" H 7900 5700 50  0001 C CNN
 F 1 "GND" H 7900 5800 50  0001 C CNN
 F 2 "" H 7900 5950 50  0000 C CNN
@@
 $EndComp
 $Comp
-L VCC #PWR016
+L VCC #PWR015
 U 1 1 5A43E812
 P 7950 3050
-F 0 "#PWR016" H 7950 2900 50  0001 C CNN
+F 0 "#PWR015" H 7950 2900 50  0001 C CNN
 F 1 "VCC" H 7950 3200 50  0000 C CNN
 F 2 "" H 7950 3050 50  0000 C CNN
@@
 $EndComp
 $Comp
-L GND #PWR017
+L GND #PWR016
 U 1 1 5A43CE5B
 P 8300 5950
-F 0 "#PWR017" H 8300 5700 50  0001 C CNN
+F 0 "#PWR016" H 8300 5700 50  0001 C CNN
 F 1 "GND" H 8300 5800 50  0001 C CNN
 F 2 "" H 8300 5950 50  0000 C CNN
@@
 08 2C 10 08 2A 2D 42 01 0A 04 82 4A 8B 50 80 02 81 A0 D2 22 14 A0 40 20 A8 B4 08 05 28 10 08 2A
 2D 42 01 0A 04 82 4A 8B AA 99 BB 25 10 08 04 02 37 21 7A 80 02 81 A0 D2 F2 FF 6C 4F 00 04 F4 D6
-7A A4 00 00 00 00 49 45 4E 44 AE 42 60 82 5D
+7A A4 00 00 00 00 49 45 4E 44 AE 42 60 82 65
 EndData
 $EndBitmap
@@
 $EndComp
 $Comp
-L GND #PWR018
+L GND #PWR017
 U 1 1 5A448571
 P 1850 7850
-F 0 "#PWR018" H 1850 7600 50  0001 C CNN
+F 0 "#PWR017" H 1850 7600 50  0001 C CNN
 F 1 "GND" H 1850 7700 50  0001 C CNN
 F 2 "" H 1850 7850 50  0000 C CNN
@@
 Connection ~ 5150 5550
 Wire Wire Line
-	6600 6250 6650 6250
-Wire Wire Line
-	6600 6350 6650 6350
-Wire Wire Line
-	6600 6450 6650 6450
+	6600 5600 6650 5600
+Wire Wire Line
+	6600 5700 6650 5700
+Wire Wire Line
+	6600 5800 6650 5800
 Wire Wire Line
 	5100 6950 5200 6950
@@
 Connection ~ 3450 6650
 Wire Wire Line
-	7100 5500 7000 5500
-Wire Wire Line
-	7000 5600 7050 5600
-Wire Wire Line
-	7050 5600 7050 5750
-Wire Wire Line
-	7000 5700 7050 5700
-Connection ~ 7050 5700
-Wire Wire Line
 	7900 5550 7900 5650

Commit message: Found error in BOM as exported from schematic. Grove connectors had wrong footprint assigned. Corrected mistake in schematic and updated netlist and BOM.
Parts:
- P2, P3: footprint Header:HEADER_M_2.54MM_1R4P_ST_AU_PTH -> Connector:PH_2.0_PTH

Commit message: Initial updates based on first build and testing.  Final updates to be pushed in subsequent commit(s).
Parts:
- added C? (x2): 1uF, Passive:0603, symbol CAP
- added Y?: Crystal_Small, symbol Crystal_Small
Changed lines of the file:
@@
 Sheet 1 1
 Title "Arduino Pro Mini mikroBUS Develepment Board"
-Date "2017-12-26"
-Rev "1.0"
+Date "2018-02-11"
+Rev "1.1"
 Comp "Casco Logix, LLC"
 Comment1 ""
@@
 B4 88 21 B0 40 20 A8 B4 08 05 28 10 08 2A 2D 42 01 0A 04 82 4A 8B 50 80 02 81 A0 D2 22 14 A0 40
 20 A8 B4 08 05 28 10 08 2A 2D AA 18 77 4B 20 10 08 04 6E 42 F4 00 05 02 41 A5 E5 FF 01 CF 93 00
-10 AA EE AF C4 00 00 00 00 49 45 4E 44 AE 42 60 82 7F
+10 AA EE AF C4 00 00 00 00 49 45 4E 44 AE 42 60 82 1F
 EndData
 $EndBitmap
@@
 Wire Notes Line
 	5500 1050 5500 1100
+$Comp
+L Crystal_Small Y?
+U 1 1 5A7FC3FF
+P 7200 3400
+F 0 "Y?" H 7200 3500 50  0000 C CNN
+F 1 "Crystal_Small" H 7200 3300 50  0000 C CNN
+F 2 "" H 7200 3400 50  0000 C CNN
+F 3 "" H 7200 3400 50  0000 C CNN
+	1    7200 3400
+	1    0    0    -1
+$EndComp
+$Comp
+L CAP C?
+U 1 1 5A7FC4B8
+P 7200 2900
+F 0 "C?" H 7260 2950 40  0000 L CNN
+F 1 "1uF" H 7260 2840 40  0000 L CNN
+F 2 "Passive:0603" H 7200 2900 60  0001 C CNN
+F 3 "" H 7200 2900 60  0000 C CNN
+	1    7200 2900
+	1    0    0    -1
+$EndComp
+$Comp
+L CAP C?
+U 1 1 5A7FC549
+P 7250 4000
+F 0 "C?" H 7310 4050 40  0000 L CNN
+F 1 "1uF" H 7310 3940 40  0000 L CNN
+F 2 "Passive:0603" H 7250 4000 60  0001 C CNN
+F 3 "" H 7250 4000 60  0000 C CNN
+	1    7250 4000
+	1    0    0    -1
+$EndComp
 $EndSCHEMATC
